File: usbc_banana_adapter.kicad_pcb (KiCad board)
At the start: 2 copper layers, 35 x 25 mm, 21 parts, among them P1 USB_C_Plug_USB2.0, SW1 DSHP02TSGER, U1 TPS25810RVCR, U3 TPS2514DBVR

Commit message: layout
Parts:
- added FID1: Fiducial, Fiducial:Fiducial_1mm_Mask2mm, F.Cu at (126.0, 69.0)
- added FID2: Fiducial, Fiducial:Fiducial_1mm_Mask2mm, F.Cu at (94.0, 69.0)
- added FID3: Fiducial, Fiducial:Fiducial_1mm_Mask2mm, F.Cu at (126.0, 91.0)
- added H5: MountingHole, MountingHole:ToolingHole_1.152mm, F.Cu at (126.0, 88.5)
- added H6: MountingHole, MountingHole:ToolingHole_1.152mm, F.Cu at (94.0, 71.5)
- P1: value USB_C_Plug_USB2.0 -> UJ20-C-V-C-3-SMT-TR
- moved R4 1.00 mm to (109.5, 91.0)
- moved U1 1.00 mm to (109.0, 87.5)
- moved C6 0.75 mm to (105.0, 70.8)
- moved U3 0.75 mm to (108.0, 70.8)
- moved C2 0.50 mm to (105.5, 89.0)
- moved C1 0.25 mm to (102.2, 89.0)
- moved C3 0.25 mm to (113.2, 85.5)
- moved C4 0.25 mm to (98.8, 89.0)
- moved C5 0.25 mm to (95.2, 89.0)
- moved D4 0.25 mm to (113.2, 88.5)
Routing:
- net /VBUS: track 0.00 -> 10.8 mm, vias 0 -> 5
- added copper zone on F.Cu, net +5V
- added copper zone on B.Cu, net /VBUS
- added copper zone on F.Cu, net GND

Commit message: layout
Parts:
- removed D2: LED_Small, LED_SMD:LED_0603_1608Metric_Pad1.05x0.95mm_HandSolder
- removed R6: 10k, Resistor_SMD:R_0603_1608Metric_Pad0.98x0.95mm_HandSolder
- added R9: 0, Resistor_SMD:R_0603_1608Metric_Pad0.98x0.95mm_HandSolder, F.Cu at (105.0, 72.5)
- moved D3 7.16 mm to (105.0, 70.0)
- moved C6 6.75 mm to (111.8, 70.5), turned to -90 degrees
- moved D1 4.03 mm to (99.0, 72.5)
- moved R5 2.12 mm to (99.0, 70.5)
- moved U3 1.03 mm to (109.0, 70.5), turned to 90 degrees
- moved R4 0.50 mm to (109.5, 90.5)
- moved U1 0.50 mm to (109.0, 87.0)
- moved D4 0.35 mm to (113.0, 88.2)
- moved R7 0.35 mm to (116.8, 91.2)
- moved R8 0.25 mm to (121.0, 91.2)
- moved SW1 0.25 mm to (120.2, 88.0)
Connections:
- C6 pad 2: Net-(U3-GND) -> GND
- D3 pad 2: /VBUS -> unconnected-(D3-K-Pad2)
- D3 pad 3: Net-(P1-D-) -> Net-(U3-DP1)
- D3 pad 4: Net-(P1-D+) -> Net-(U3-DM1)
- D4 pad 2: Net-(P1-VCONN) -> /VBUS
- D4 pad 4: unconnected-(D4-K-Pad4) -> Net-(P1-CC2)
- P1 pad A6: Net-(P1-D+) -> Net-(U3-DP1)
- P1 pad A7: Net-(P1-D-) -> Net-(U3-DM1)
- P1 pad A8: (no net) -> unconnected-(P1-SBU1-PadA8)
- P1 pad B5: Net-(P1-VCONN) -> Net-(P1-CC2)
- P1 pad B6: (no net) -> Net-(U3-DP1)
- P1 pad B7: (no net) -> Net-(U3-DM1)
- P1 pad B8: (no net) -> unconnected-(P1-SBU2-PadB8)
- U1 pad 13: Net-(P1-VCONN) -> Net-(P1-CC2)
- U1 pad 20: Net-(D2-K) -> unconnected-(U1-~{LD_DET}-Pad20)
- U3 pad 1: Net-(P1-D+) -> Net-(U3-DP1)
- U3 pad 2: Net-(U3-GND) -> GND
- U3 pad 6: Net-(P1-D-) -> Net-(U3-DM1)
Routing:
- net +5V: track 0.00 -> 49.0 mm, vias 0 -> 3
- net GND: track 0.00 -> 39.3 mm, vias 0 -> 17
- net Net-(P1-CC2): track 0.00 -> 31.4 mm, vias 0 -> 2
- net Net-(U1-CHG_HI): track 0.00 -> 21.4 mm
- net Net-(P1-CC1): track 0.00 -> 21.0 mm, vias 0 -> 1
- net Net-(U3-DP1): track 0.00 -> 19.8 mm, vias 0 -> 2
- net Net-(U1-CHG): track 0.00 -> 18.9 mm
- net Net-(D1-K): track 0.00 -> 18.2 mm
- net Net-(U3-DM1): track 0.00 -> 14.3 mm
- net /VBUS: track 10.8 -> 24.9 mm
- net Net-(D1-A): track 0.00 -> 2.74 mm
- net Net-(U1-REF_RTN): track 0.00 -> 1.87 mm
- net Net-(U1-REF): track 0.00 -> 1.87 mm
- added copper zone on F.Cu, net /VBUS

Commit message: revA ready
Parts:
- added C7: 47uF, Capacitor_SMD:C_1206_3216Metric_Pad1.33x1.80mm_HandSolder, F.Cu at (96.5, 73.0)
- C1, C4, C5: footprint Capacitor_SMD:C_1210_3225Metric_Pad1.33x2.70mm_HandSolder -> Capacitor_SMD:C_1206_3216Metric_Pad1.33x1.80mm_HandSolder
- D1: value LED_Small -> KT-0603R
- SW1: value DSHP02TSGER -> DSHP02TJGER; footprint Button_Switch_SMD:SW_DIP_SPSTx02_Slide_KingTek_DSHP02TS_W7.62mm_P1.27mm -> Button_Switch_SMD:SW_DIP_SPSTx02_Slide_KingTek_DSHP02TJ_W5.25mm_P1.27mm_JPin
- moved H6 4.72 mm to (98.0, 69.0)
- moved R8 4.50 mm to (116.5, 91.2), turned to 0 degrees
- moved R7 4.00 mm to (120.8, 91.2), turned to 180 degrees
- moved D1 2.00 mm to (101.0, 72.5)
- moved R5 2.00 mm to (101.0, 70.5)
- moved FID1 1.50 mm to (124.5, 69.0)
- moved FID2 1.50 mm to (95.5, 69.0)
- moved FID3 1.50 mm to (124.5, 91.0)
- moved H5 1.50 mm to (124.5, 88.5)
- moved C5 1.25 mm to (96.5, 89.0)
- moved C4 1.00 mm to (99.8, 89.0)
- moved SW1 0.79 mm to (119.5, 87.8)
- moved C1 0.75 mm to (103.0, 89.0)
Connections:
- R7 pad 1: +5V -> Net-(U1-CHG_HI)
- R7 pad 2: Net-(U1-CHG) -> GND
- R8 pad 1: +5V -> Net-(U1-CHG)
- R8 pad 2: Net-(U1-CHG_HI) -> GND
- SW1 pad 1: GND -> +5V
- SW1 pad 2: GND -> +5V
Routing:
- net GND: track 39.3 -> 51.9 mm
- net Net-(U1-CHG_HI): track 21.4 -> 23.7 mm
- net Net-(D1-K): track 18.2 -> 16.2 mm
- net Net-(U1-CHG): track 18.9 -> 17.3 mm
- net +5V: track 49.0 -> 50.0 mm, vias 3 -> 2
Other:
- board size 35 x 25 mm -> 32 x 25 mm
- board text added: "C"
- board text added: "CH"
- board text added: "USB-C DFP USB BC1.2 Rev A 4V5 - 5V5 / 3A Max SET SW1 TO ADJ ILIM"
- board text removed: "-"
- board text removed: "USB-C 1.2 DFP USB BC1.2 Rev A"

Commit message: swap banana
Parts:
- moved C1 9.60 mm to (109.0, 96.5)
- moved C2 9.60 mm to (111.5, 96.5)
- moved C3 9.60 mm to (119.2, 93.0)
- moved C4 9.60 mm to (105.8, 96.5)
- moved C5 9.60 mm to (102.5, 96.5)
- moved C6 9.60 mm to (117.8, 78.0)
- moved C7 9.60 mm to (102.5, 80.5)
- moved D1 9.60 mm to (107.0, 80.0)
- moved D3 9.60 mm to (111.0, 77.5)
- moved D4 9.60 mm to (119.0, 95.8)
- moved FID1 9.60 mm to (130.5, 76.5)
- moved FID2 9.60 mm to (101.5, 76.5)
- moved FID3 9.60 mm to (130.5, 98.5)
- moved H1 9.60 mm to (106.5, 87.5)
- moved H2 9.60 mm to (125.5, 87.5)
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Other:
- board text added: "-"

Commit message: tweak via size
Routing:
- net GND: vias 17 -> 20
Changed lines of the file:
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@@
 	)
 	(via
-		(at 115 94.5)
-		(size 0.6)
-		(drill 0.3)
+		(at 114.5 94.5)
+		(size 0.5)
+		(drill 0.2)
 		(layers "F.Cu" "B.Cu")
 		(free yes)
@@
 	)
 	(via
-		(at 115 93.5)
-		(size 0.6)
-		(drill 0.3)
+		(at 114.5 93.5)
+		(size 0.5)
+		(drill 0.2)
 		(layers "F.Cu" "B.Cu")
 		(free yes)
@@
 	)
 	(via
-		(at 115 95.5)
-		(size 0.6)
-		(drill 0.3)
+		(at 115.5 95.5)
+		(size 0.5)
+		(drill 0.2)
+		(layers "F.Cu" "B.Cu")
+		(free yes)
+		(net "GND")
+	)
+	(via
+		(at 114.5 95.5)
+		(size 0.5)
+		(drill 0.2)
 		(layers "F.Cu" "B.Cu")
 		(free yes)
@@
 	)
 	(via
+		(at 115.5 93.5)
+		(size 0.5)
+		(drill 0.2)
+		(layers "F.Cu" "B.Cu")
+		(free yes)
+		(net "GND")
+	)
+	(via
 		(at 101.5 80)
 		(size 0.6)
@@
 		(layers "F.Cu" "B.Cu")
 		(free yes)
+		(net "GND")
+	)
+	(via
+		(at 115.5 94.5)
+		(size 0.5)
+		(drill 0.2)
+		(layers "F.Cu" "B.Cu")
+		(free yes)
